File: PCB/RevC/kas_mam.kicad_pcb (KiCad board)
At the start: 2 copper layers, 100 x 100 mm, 201 parts, among them K1 5V-relay, P4 CONN_02X20, Q1 BC857, Q10 BC547, Q11 BC547, Q12 BC547, Q13 DB241C, Q14 DB241C, Q15 DB241C, Q16 DB241C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

Commit message: RevC v 1.1
Fis for PCB. Should work now.
Parts:
- moved C2 0.75 mm to (67.7, 59.3)
- moved C3 0.75 mm to (74.5, 59.3)
- moved U3 0.60 mm to (71.2, 64.9)
Connections:
- U3 pad 1: +3V3 -> (no net)
- U3 pad 14: (no net) -> /5PI_MOSI
- U3 pad 15: /5PI_MOSI -> /5PI_MISO
- U3 pad 16: /5PI_MISO -> /INT
- U3 pad 17: /INT -> /5PI_CLK
- U3 pad 18: /5PI_CLK -> /5PI_CS0
- U3 pad 19: /5PI_CS0 -> +5V
- U3 pad 2: /SPI_CS0 -> +3V3
- U3 pad 20: +5V -> (no net)
- U3 pad 3: /SPI_CLK -> /SPI_CS0
- U3 pad 4: /27 -> /SPI_CLK
- U3 pad 5: /SPI_MISO -> /27
- U3 pad 6: /SPI_MOSI -> /SPI_MISO
- U3 pad 7: (no net) -> /SPI_MOSI
- U7 pad 1: +3V3 -> /Pi_flow1
- U7 pad 19: /Flow_sen1 -> +5V
- U7 pad 2: /Pi_flow1 -> +3V3
- U7 pad 20: +5V -> /Flow_sen1
Routing:
- net GND: track 239.1 -> 296.2 mm
- net +5V: track 387.6 -> 393.2 mm, vias 14 -> 16
- net +3V3: track 135.9 -> 139.5 mm, vias 4 -> 5
- net /Flow_sen1: track 12.7 -> 13.6 mm
- net /INT: track 64.8 -> 64.0 mm
- net /PI_SDA: track 66.0 -> 65.4 mm
- net /Pi_flow1: track 13.8 -> 14.3 mm
Other:
- board text added: "v1.1"
