File: PCB/RevC/kas_mam.sch (KiCad schematic (older format))
At the start: 197 parts, among them K1 5V-relay, P4 CONN_02X20, Q1 BC857, Q10 BC547, Q11 BC547, Q12 BC547, Q13 DB241C, Q14 DB241C, Q15 DB241C, Q16 DB241C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

Commit message: RevC v 1.1
Fis for PCB. Should work now.
Connections:
- net +3V3: now also U3.2 (Va), U7.2 (Va); no longer U3.1 (A1), U7.1 (A1)
- net +5V: now also U3.19 (Vb), U7.19 (Vb); no longer U3.20 (B1), U7.20 (B1)
- net 27: now also U3.5 (A4); no longer U3.4 (A3)
- net 5PI_CLK: now also U3.17 (B3); no longer U3.18 (B2)
- net 5PI_CS0: now also U3.18 (B2); no longer U3.19 (Vb)
- net 5PI_MISO: now also U3.15 (B5); no longer U3.16 (B4)
- net 5PI_MOSI: now also U3.14 (B6); no longer U3.15 (B5)
- net Flow_sen1: now also U7.20 (B1); no longer U7.19 (Vb)
- net INT: now also U3.16 (B4); no longer U3.17 (B3)
- net Pi_flow1: now also U7.1 (A1); no longer U7.2 (Va)
- net SPI_CLK: now also U3.4 (A3); no longer U3.3 (A2)
- net SPI_CS0: now also U3.3 (A2); no longer U3.2 (Va)
- net SPI_MISO: now also U3.6 (A5); no longer U3.5 (A4)
- net SPI_MOSI: now also U3.7 (A6); no longer U3.6 (A5)
- no-connect marks 25 -> 29
Other:
- moved on the sheet: C2, C3, C4, C5
