File: PCB/PSU/PSU.kicad_pcb (KiCad board)
At the start: 2 copper layers, 125 x 100 mm, 144 parts, among them J1 Conn_01x02, J10 Conn_01x03, J11 Conn_01x01, J12 Conn_01x02, J13 Conn_01x02, J14 Conn_01x03, J15 Conn_01x03, J16 Conn_01x01, J17 Conn_01x02, J18 Conn_01x04, J19 Conn_01x04, J2 Conn_01x04, J3 Conn_01x03, J4 Conn_01x04, J5 Conn_01x01, J6 Conn_01x02, J7 Conn_01x03, J8 Conn_01x01, J9 Conn_01x02, Q1 BD139, Q2 BD139, Q3 BD139, Q4 BC847, Q5 BD139, Q6 BC847, Q7 BC847, Q8 BC847, Q9 BC847, U1 LM7805CT, U10 DS18B20, U11 LM317_3PinPackage, U12 MCP23008, U2 LM7812CT, U3 LM7805CT, U4 LM7812CT, U5 INA219, U6 INA219, U7 LM317_3PinPackage, U8 LM317_3PinPackage, U9 LM317_3PinPackage

Commit message: PSU PCB rev A final
Parts:
- moved R31 5.77 mm to (112.5, 64.0), turned to 0 degrees
- moved R32 5.76 mm to (112.5, 66.2), turned to 180 degrees
Connections:
- J17 pad 1: /SDA -> /CSL
- J17 pad 2: /CSL -> /SDA
- R31 pad 2: /SDA -> /CSL
- R32 pad 1: /CSL -> /SDA
- U5 pad 1: +5V -> /5Vout
- U5 pad 2: /5Vout -> +5V
- U6 pad 1: +12V -> /12Vout
- U6 pad 2: /12Vout -> +12V
Routing:
- net Net-(J13-Pad2): track 61.9 -> 48.3 mm
- net /12Vout: track 108.3 -> 96.8 mm
- net +5V: track 149.9 -> 159.4 mm, vias 10 -> 8
- net +12V: track 245.3 -> 236.7 mm
- net Net-(J6-Pad2): track 95.2 -> 90.4 mm
- net GND: track 280.5 -> 277.8 mm
- net /3.3v: track 74.0 -> 72.0 mm
- net /Tdata: track 71.7 -> 69.9 mm
- net /5Vout: track 84.4 -> 85.6 mm
- net /LED4: track 59.7 -> 60.8 mm
- net /CSL: track 67.6 -> 66.8 mm, vias 5 -> 6
- net /SDA: track 65.3 -> 65.0 mm, vias 7 -> 6
Other:
- board text added: "15-25VAC"
- board text removed: "15-25VAC in"
