File: PCB/PSU/PSU.sch (KiCad schematic (older format))
At the start: 140 parts, among them J1 Conn_01x02, J10 Conn_01x03, J11 Conn_01x01, J12 Conn_01x02, J13 Conn_01x02, J14 Conn_01x03, J15 Conn_01x03, J16 Conn_01x01, J17 Conn_01x02, J18 Conn_01x04, J19 Conn_01x04, J2 Conn_01x04, J3 Conn_01x03, J4 Conn_01x04, J5 Conn_01x01, J6 Conn_01x02, J7 Conn_01x03, J8 Conn_01x01, J9 Conn_01x02, Q1 BD139, Q2 BD139, Q3 BD139, Q4 BC847, Q5 BD139, Q6 BC847, Q7 BC847, Q8 BC847, Q9 BC847, U1 LM7805CT, U10 DS18B20, U11 LM317_3PinPackage, U12 MCP23008, U2 LM7812CT, U3 LM7805CT, U4 LM7812CT, U5 INA219, U6 INA219, U7 LM317_3PinPackage, U8 LM317_3PinPackage, U9 LM317_3PinPackage

Commit message: PSU PCB rev A final
Connections:
- net +12V: now also U6.2 (IN-); no longer U6.1 (IN+)
- net +5V: now also U5.2 (IN-); no longer U5.1 (IN+)
- net 12Vout: now also U6.1 (IN+); no longer U6.2 (IN-)
- net 5Vout: now also U5.1 (IN+); no longer U5.2 (IN-)
- net CSL: now also J17.1 (Pin_1), R31.2; no longer J17.2 (Pin_2), R32.1
- net SDA: now also J17.2 (Pin_2), R32.1; no longer J17.1 (Pin_1), R31.2
Other:
- moved on the sheet: R1, R2
Changed lines of the file:
@@
 L +12V #PWR01
 U 1 1 59A7360D
-P 8050 3600
-F 0 "#PWR01" H 8050 3450 50  0001 C CNN
-F 1 "+12V" H 8050 3740 50  0000 C CNN
-F 2 "" H 8050 3600 50  0000 C CNN
-F 3 "" H 8050 3600 50  0000 C CNN
-	1    8050 3600
+P 8050 3400
+F 0 "#PWR01" H 8050 3250 50  0001 C CNN
+F 1 "+12V" H 8050 3540 50  0000 C CNN
+F 2 "" H 8050 3400 50  0000 C CNN
+F 3 "" H 8050 3400 50  0000 C CNN
+	1    8050 3400
 	0    1    1    0
 $EndComp
@@
 L R_Small R1
 U 1 1 59A7DE44
-P 7850 1500
-F 0 "R1" H 7880 1520 50  0000 L CNN
-F 1 "0R04" H 7880 1460 50  0000 L CNN
-F 2 "Resistors_SMD:R_2512_HandSoldering" H 7850 1500 50  0001 C CNN
-F 3 "" H 7850 1500 50  0000 C CNN
-	1    7850 1500
-	0    -1   -1   0
+P 7950 1400
+F 0 "R1" H 7980 1420 50  0000 L CNN
+F 1 "0R04" H 7980 1360 50  0000 L CNN
+F 2 "Resistors_SMD:R_2512_HandSoldering" H 7950 1400 50  0001 C CNN
+F 3 "" H 7950 1400 50  0000 C CNN
+	1    7950 1400
+	-1   0    0    1
 $EndComp
 $Comp
@@
 L +5V #PWR06
 U 1 1 59A7EE54
-P 7950 1500
-F 0 "#PWR06" H 7950 1350 50  0001 C CNN
-F 1 "+5V" H 7950 1640 50  0000 C CNN
-F 2 "" H 7950 1500 50  0000 C CNN
-F 3 "" H 7950 1500 50  0000 C CNN
-	1    7950 1500
+P 8050 1300
+F 0 "#PWR06" H 8050 1150 50  0001 C CNN
+F 1 "+5V" H 8050 1440 50  0000 C CNN
+F 2 "" H 8050 1300 50  0000 C CNN
+F 3 "" H 8050 1300 50  0000 C CNN
+	1    8050 1300
 	0    1    1    0
 $EndComp
@@
 L R_Small R2
 U 1 1 59A8C52C
-P 7850 3600
-F 0 "R2" H 7880 3620 50  0000 L CNN
-F 1 "0R04" H 7880 3560 50  0000 L CNN
-F 2 "Resistors_SMD:R_2512_HandSoldering" H 7850 3600 50  0001 C CNN
-F 3 "" H 7850 3600 50  0000 C CNN
-	1    7850 3600
-	0    -1   -1   0
+P 7950 3500
+F 0 "R2" H 7980 3520 50  0000 L CNN
+F 1 "0R04" H 7980 3460 50  0000 L CNN
+F 2 "Resistors_SMD:R_2512_HandSoldering" H 7950 3500 50  0001 C CNN
+F 3 "" H 7950 3500 50  0000 C CNN
+	1    7950 3500
+	-1   0    0    1
 $EndComp
 $Comp
@@
 	2550 4150 2850 4150
 Wire Wire Line
-	3400 3600 7850 3600
+	3400 3600 7950 3600
 Connection ~ 4350 3600
 Connection ~ 6600 3600
@@
 	1    0    0    -1
 $EndComp
+Text Label 7500 5600 0    60   ~ 0
+SDA
+Wire Wire Line
+	7350 5500 7700 5500
 Text Label 7500 5500 0    60   ~ 0
-SDA
-Wire Wire Line
-	7350 5500 7700 5500
-Text Label 7500 5600 0    60   ~ 0
 CSL
 Wire Wire Line
@@
 $EndComp
 Wire Wire Line
-	7950 1650 7950 1500
-Wire Wire Line
-	3400 1500 7850 1500
-Wire Wire Line
-	7850 1500 7850 1650
-Connection ~ 7750 1500
+	7950 1500 7950 1650
+Wire Wire Line
+	3400 1500 7950 1500
 Wire Wire Line
 	7750 2750 7750 2550
@@
 Connection ~ 7350 1800
 Wire Wire Line
-	7950 3750 7950 3600
-Wire Wire Line
-	7850 3600 7850 3750
-Connection ~ 7750 3600
+	7950 3600 7950 3750
 $Comp
 L GND #PWR052
@@
 $EndComp
 Wire Wire Line
-	7950 3600 8050 3600
-Wire Wire Line
 	7200 3700 7750 3700
 Wire Wire Line
@@
 $EndComp
 Connection ~ 9700 4500
+Wire Wire Line
+	7850 1650 7850 1300
+Wire Wire Line
+	7850 1300 8050 1300
+Connection ~ 7950 1300
+Wire Wire Line
+	7850 3750 7850 3400
+Wire Wire Line
+	7850 3400 8050 3400
+Connection ~ 7950 3400
 $EndSCHEMATC
