File: PCB/MainBoard/kas_mam.kicad_pcb (KiCad board)
At the start: 2 copper layers, 100 x 100 mm, 201 parts, among them K1 5V-relay, P4 CONN_02X20, Q1 BC857, Q10 BC547, Q11 BC547, Q12 BC547, Q13 DB241C, Q14 DB241C, Q15 DB241C, Q16 DB241C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

Commit message: Main Board rev D
Parts:
- added GPIO1: CONN_01X02, Pin_Headers:Pin_Header_Straight_1x02_Pitch2.54mm, F.Cu at (90.0, 101.0)
- added i2c1: CONN_01X02, Connectors_Molex:Molex_KK-6410-02_02x2.54mm_Straight, F.Cu at (83.0, 101.0)
- Q1, Q2, Q3: value BC857 -> BC847
- moved U4 1.50 mm to (81.5, 92.0)
- moved C3 0.40 mm to (74.8, 59.3), turned to 0 degrees
- moved LCD1 0.15 mm to (58.2, 52.0)
- moved C2 0.07 mm to (67.8, 59.3), turned to 0 degrees
- turned Q2 to 270 degrees
- renumbered REF** to ?
Connections:
- P4 pad 17: (no net) -> /24
- P4 pad 21: /27 -> /25
- Q1 pad 2: +5V -> Net-(LCD1-Pad7)
- Q1 pad 3: Net-(LCD1-Pad7) -> +5V
- Q2 pad 2: Net-(D1-Pad1) -> +5V
- Q2 pad 3: +5V -> Net-(D1-Pad1)
- Q3 pad 2: +5V -> Net-(Q3-Pad2)
- Q3 pad 3: Net-(Q3-Pad3) -> +5V
- STATUS1 pad 1: Net-(Q3-Pad3) -> Net-(Q3-Pad2)
- U3 pad 1: (no net) -> /SPI_CS0
- U3 pad 12: /I2C_SDA -> /INTu4
- U3 pad 13: /I2C_CSL -> /I2C_SDA
- U3 pad 14: /5PI_MOSI -> /I2C_CSL
- U3 pad 15: /5PI_MISO -> /5PI_MOSI
- U3 pad 16: /INT -> /5PI_MISO
- U3 pad 17: /5PI_CLK -> /INTu5
- U3 pad 18: /5PI_CS0 -> /5PI_CLK
- U3 pad 20: (no net) -> /5PI_CS0
- U3 pad 3: /SPI_CS0 -> /SPI_CLK
- U3 pad 4: /SPI_CLK -> /25
- U3 pad 5: /27 -> /SPI_MISO
- U3 pad 6: /SPI_MISO -> /SPI_MOSI
- U3 pad 7: /SPI_MOSI -> /PI_SCL
- U3 pad 8: /PI_SCL -> /PI_SDA
- U3 pad 9: /PI_SDA -> /24
- U4 pad 1: Net-(R83-Pad2) -> Net-(GPIO1-Pad2)
- U4 pad 2: Net-(R84-Pad2) -> Net-(GPIO1-Pad1)
- U4 pad 20: (no net) -> /INTu4
- U4 pad 3: Net-(R85-Pad2) -> Net-(R83-Pad2)
- U4 pad 4: Net-(R86-Pad2) -> Net-(R84-Pad2)
- U4 pad 5: Net-(R87-Pad2) -> Net-(R85-Pad2)
- U4 pad 6: Net-(R88-Pad2) -> Net-(R86-Pad2)
- U4 pad 7: (no net) -> Net-(R87-Pad2)
- U4 pad 8: (no net) -> Net-(R88-Pad2)
- U5 pad 20: /INT -> /INTu5
Routing:
- net /INTu5: track 0.00 -> 64.3 mm, vias 0 -> 3
- net /INT: track 64.0 -> 0.00 mm, vias 3 -> 0
- net /INTu4: track 0.00 -> 51.2 mm, vias 0 -> 4
- net /24: track 0.00 -> 47.4 mm, vias 0 -> 1
- net /27: track 46.2 -> 0.00 mm
- net /25: track 0.00 -> 46.2 mm
- net /I2C_CSL: track 90.0 -> 114.3 mm, vias 4 -> 6
- net /I2C_SDA: track 91.6 -> 113.0 mm, vias 4 -> 5
- net Net-(GPIO1-Pad1): track 0.00 -> 15.2 mm, vias 0 -> 2
- net Net-(GPIO1-Pad2): track 0.00 -> 14.9 mm, vias 0 -> 2
- net GND: track 296.2 -> 303.8 mm
- net +3V3: track 139.5 -> 145.5 mm
- net Net-(R83-Pad2): track 81.1 -> 75.2 mm
- net Net-(R84-Pad2): track 76.2 -> 70.5 mm
- net Net-(Q3-Pad3): track 5.59 -> 0.00 mm
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Other:
- board text added: "rev.D"
- board text removed: "rev.C"
- board text removed: "v1.1"
