File: PCB/MainBoard/kas_mam.sch (KiCad schematic (older format))
At the start: 197 parts, among them K1 5V-relay, P4 CONN_02X20, Q1 BC857, Q10 BC547, Q11 BC547, Q12 BC547, Q13 DB241C, Q14 DB241C, Q15 DB241C, Q16 DB241C, Q17 DB241C, Q2 BC857, Q3 BC857, Q4 BC547, Q5 BC547, Q6 DB241C, Q7 DB241C, Q8 BC547, Q9 BC547, SW1 SW_PUSH, SW2 SW_PUSH, U1 MCP3208, U2 MCP23017, U3 TXS0108E, U4 MCP23017, U5 MCP23017, U6 MCP23017, U7 TXS0108E

Commit message: Main Board rev D
Parts:
- removed Q1, Q2, Q3: BC857, TO_SOT_Packages_SMD:SOT-23, symbol BC857
- added GPIO1: CONN_01X02, Pin_Headers:Pin_Header_Straight_1x02_Pitch2.54mm, symbol CONN_01X02
- added Q1, Q2, Q3: BC847, TO_SOT_Packages_SMD:SOT-23, symbol BC847
- added i2c1: CONN_01X02, Connectors_Molex:Molex_KK-6410-02_02x2.54mm_Straight, symbol CONN_01X02
- D10, D11, D12, D13, D14, D15, D16, D17, D18, D19, D2, D20, D21, D22, D23, D24, D25, D26, D27, D28, D29, D3, D30, D31, D32, D33, D34, D35, D36, D37, D4, D5, D6, D7, D8, D9: symbol LED -> LED-RESCUE-kas_mam
- RV1: symbol POT -> POT-RESCUE-kas_mam
- U1: symbol MCP3208 -> MCP3208-RESCUE-kas_mam
- U2, U4, U5, U6: symbol MCP23017 -> MCP23017-RESCUE-kas_mam
Connections:
- net labels added: 24, 25, INTu4, INTu5
- net labels removed: 27, INT, blah
- wire segments 501 -> 508
- no-connect marks 29 -> 23
Other:
- moved on the sheet: R83, R84, R85, R86, R87, R88
